Commit message: Update GR3

File: openrd/urdf/fourier_gr3/gr3.urdf (robot description, URDF)
Before this commit: robot gr3, 37 links, 36 joints
Links:
- added link L_hand_base_link, mass 0.29928; collision mesh filename=../meshes/fourier_hand_6dof/L_hand_base_link.STL; visual mesh filename=../meshes/fourier_hand_6dof/L_hand_base_link.STL
- added link L_index_intermediate_link, mass 0.0027085; collision mesh filename=../meshes/fourier_hand_6dof/L_index_intermediate_link.STL; visual mesh filename=../meshes/fourier_hand_6dof/L_index_intermediate_link.STL
- added link L_index_proximal_link, mass 0.011244; collision mesh filename=../meshes/fourier_hand_6dof/L_index_proximal_link.STL; visual mesh filename=../meshes/fourier_hand_6dof/L_index_proximal_link.STL
- added link L_index_tip_link; visual sphere radius=0.005
- added link L_middle_intermediate_link, mass 0.0032739; collision mesh filename=../meshes/fourier_hand_6dof/L_middle_intermediate_link.STL; visual mesh filename=../meshes/fourier_hand_6dof/L_middle_intermediate_link.STL
- added link L_middle_proximal_link, mass 0.011244; collision mesh filename=../meshes/fourier_hand_6dof/L_middle_proximal_link.STL; visual mesh filename=../meshes/fourier_hand_6dof/L_middle_proximal_link.STL
- added link L_middle_tip_link; visual sphere radius=0.005
- added link L_pinky_intermediate_link, mass 0.0024076; collision mesh filename=../meshes/fourier_hand_6dof/L_pinky_intermediate_link.STL; visual mesh filename=../meshes/fourier_hand_6dof/L_pinky_intermediate_link.STL
- added link L_pinky_proximal_link, mass 0.011244; collision mesh filename=../meshes/fourier_hand_6dof/L_pinky_proximal_link.STL; visual mesh filename=../meshes/fourier_hand_6dof/L_pinky_proximal_link.STL
- added link L_pinky_tip_link; visual sphere radius=0.005
- added link L_ring_intermediate_link, mass 0.0027085; collision mesh filename=../meshes/fourier_hand_6dof/L_ring_intermediate_link.STL; visual mesh filename=../meshes/fourier_hand_6dof/L_ring_intermediate_link.STL
- added link L_ring_proximal_link, mass 0.011244; collision mesh filename=../meshes/fourier_hand_6dof/L_ring_proximal_link.STL; visual mesh filename=../meshes/fourier_hand_6dof/L_ring_proximal_link.STL
- added link L_ring_tip_link; visual sphere radius=0.005
- added link L_thumb_distal_link, mass 0.018024; collision mesh filename=../meshes/fourier_hand_6dof/L_thumb_distal_link.STL; visual mesh filename=../meshes/fourier_hand_6dof/L_thumb_distal_link.STL
- added link L_thumb_proximal_pitch_link, mass 0.060766; collision mesh filename=../meshes/fourier_hand_6dof/L_thumb_proximal_pitch_link.STL; visual mesh filename=../meshes/fourier_hand_6dof/L_thumb_proximal_pitch_link.STL
- added link L_thumb_proximal_yaw_link, mass 0.0084328; collision mesh filename=../meshes/fourier_hand_6dof/L_thumb_proximal_yaw_link.STL; visual mesh filename=../meshes/fourier_hand_6dof/L_thumb_proximal_yaw_link.STL
- added link L_thumb_tip_link; visual sphere radius=0.005
- added link R_hand_base_link, mass 0.2993; collision mesh filename=../meshes/fourier_hand_6dof/R_hand_base_link.STL; visual mesh filename=../meshes/fourier_hand_6dof/R_hand_base_link.STL
- added link R_index_intermediate_link, mass 0.0027085; collision mesh filename=../meshes/fourier_hand_6dof/R_index_intermediate_link.STL; visual mesh filename=../meshes/fourier_hand_6dof/R_index_intermediate_link.STL
- added link R_index_proximal_link, mass 0.011244; collision mesh filename=../meshes/fourier_hand_6dof/R_index_proximal_link.STL; visual mesh filename=../meshes/fourier_hand_6dof/R_index_proximal_link.STL
- added link R_index_tip_link; visual sphere radius=0.005
- added link R_middle_intermediate_link, mass 0.0032739; collision mesh filename=../meshes/fourier_hand_6dof/R_middle_intermediate_link.STL; visual mesh filename=../meshes/fourier_hand_6dof/R_middle_intermediate_link.STL
- added link R_middle_proximal_link, mass 0.011244; collision mesh filename=../meshes/fourier_hand_6dof/R_middle_proximal_link.STL; visual mesh filename=../meshes/fourier_hand_6dof/R_middle_proximal_link.STL
- added link R_middle_tip_link; visual sphere radius=0.005
- added link R_pinky_intermediate_link, mass 0.0024076; collision mesh filename=../meshes/fourier_hand_6dof/R_pinky_intermediate_link.STL; visual mesh filename=../meshes/fourier_hand_6dof/R_pinky_intermediate_link.STL
- added link R_pinky_proximal_link, mass 0.011244; collision mesh filename=../meshes/fourier_hand_6dof/R_pinky_proximal_link.STL; visual mesh filename=../meshes/fourier_hand_6dof/R_pinky_proximal_link.STL
- added link R_pinky_tip_link; visual sphere radius=0.005
- added link R_ring_intermediate_link, mass 0.0027085; collision mesh filename=../meshes/fourier_hand_6dof/R_ring_intermediate_link.STL; visual mesh filename=../meshes/fourier_hand_6dof/R_ring_intermediate_link.STL
- added link R_ring_proximal_link, mass 0.011244; collision mesh filename=../meshes/fourier_hand_6dof/R_ring_proximal_link.STL; visual mesh filename=../meshes/fourier_hand_6dof/R_ring_proximal_link.STL
- added link R_ring_tip_link; visual sphere radius=0.005
- added link R_thumb_distal_link, mass 0.018024; collision mesh filename=../meshes/fourier_hand_6dof/R_thumb_distal_link.STL; visual mesh filename=../meshes/fourier_hand_6dof/R_thumb_distal_link.STL
- added link R_thumb_proximal_pitch_link, mass 0.060766; collision mesh filename=../meshes/fourier_hand_6dof/R_thumb_proximal_pitch_link.STL; visual mesh filename=../meshes/fourier_hand_6dof/R_thumb_proximal_pitch_link.STL
- added link R_thumb_proximal_yaw_link, mass 0.0084327; collision mesh filename=../meshes/fourier_hand_6dof/R_thumb_proximal_yaw_link.STL; visual mesh filename=../meshes/fourier_hand_6dof/R_thumb_proximal_yaw_link.STL
- added link R_thumb_tip_link; visual sphere radius=0.005
- link base_link: mass 6.2879 -> 6.19011858
- link camera_link: mass None -> 0.00156615; geometry visual mesh filename=../../meshes/fourier_gr3/camera_link.STL
- link imu_link: mass 0.05 -> 0.03
- link left_foot_pitch_link: mass 0.099137 -> 0.0594926
- link left_foot_roll_link: mass 1.1598 -> 1.21412398
- link left_hand_pitch_link: mass 0.55738 -> 0.57735702
- link left_hand_roll_link: mass 0.20757 -> 0.2121397
- link left_hand_yaw_link: mass 1.2082 -> 1.21478268
- link left_lower_arm_pitch_link: mass 0.86582 -> 0.87226659
- link left_shank_pitch_link: mass 3.0159 -> 3.19509257
- link left_thigh_pitch_link: mass 2.0188 -> 2.11064201
- link left_thigh_roll_link: mass 3.2696 -> 3.23888801
- link left_thigh_yaw_link: mass 6.1825 -> 5.4181897
- link left_upper_arm_pitch_link: mass 1.358 -> 1.40210533
- link left_upper_arm_roll_link: mass 1.3091 -> 1.14984334
- link left_upper_arm_yaw_link: mass 1.0887 -> 1.09369321
- link right_foot_pitch_link: mass 0.099137 -> 0.0594926; geometry collision cylinder length=0.24 radius=0.02; collision cylinder length=0.24 radius=0.02
- link right_foot_roll_link: mass 1.1598 -> 1.21412398; geometry visual mesh filename=../../meshes/fourier_gr3/right_foot_roll_link.STL
- link right_hand_pitch_link: mass 0.55738 -> 0.57735702
- link right_hand_roll_link: mass 0.20757 -> 0.2121397
- link right_hand_yaw_link: mass 1.2082 -> 1.21478268
- link right_lower_arm_pitch_link: mass 0.86582 -> 0.87226659
- link right_shank_pitch_link: mass 3.0159 -> 3.19509257
- link right_thigh_pitch_link: mass 2.0188 -> 2.11064201
- link right_thigh_roll_link: mass 3.2696 -> 3.23888801
- link right_thigh_yaw_link: mass 6.1825 -> 5.4181897
- link right_upper_arm_pitch_link: mass 1.358 -> 1.40210533
- link right_upper_arm_roll_link: mass 1.3091 -> 1.14984334
- link right_upper_arm_yaw_link: mass 1.0887 -> 1.09369321
- link waist_pitch_link: mass 3.0924 -> 2.88081135
- link waist_roll_link: mass 0.165 -> 0.20486665
- link waist_yaw_link: mass 1.5935 -> 1.7648565
Joints:
- added joint L_hand_base_joint: type fixed, parent left_end_effector_link, child L_hand_base_link, origin xyz=0 0 0 rpy=0 0 0
- added joint L_index_intermediate_joint: type revolute, parent L_index_proximal_link, child L_index_intermediate_link, origin xyz=0.031533 -0.0054444 0 rpy=0 0.00014037 -0.0018338, axis 0 0 1, limit lower=-1.791 upper=0 effort=0 velocity=0, mimic joint=L_index_proximal_joint multiplier=0.975 offset=0
- added joint L_index_proximal_joint: type revolute, parent L_hand_base_link, child L_index_proximal_link, origin xyz=0.026868 -0.0123 -0.093989 rpy=0 1.5184 0, axis 0 0 1, limit lower=-1.602 upper=0 effort=0 velocity=0
- added joint L_index_tip_joint: type fixed, parent L_index_intermediate_link, child L_index_tip_link, origin xyz=0.0390 -0.0020 0 rpy=0 0 0
- added joint L_middle_intermediate_joint: type revolute, parent L_middle_proximal_link, child L_middle_intermediate_link, origin xyz=0.031521 -0.0055139 0 rpy=0 0.00015517 0.0048744, axis 0 0 1, limit lower=-1.791 upper=0 effort=0 velocity=0, mimic joint=L_middle_proximal_joint multiplier=0.975 offset=0
- added joint L_middle_proximal_joint: type revolute, parent L_hand_base_link, child L_middle_proximal_link, origin xyz=0.0085 -0.0123 -0.095992 rpy=0 1.5708 0, axis 0 0 1, limit lower=-1.603 upper=0 effort=0 velocity=0
- added joint L_middle_tip_joint: type fixed, parent L_middle_intermediate_link, child L_middle_tip_link, origin xyz=0.047 -0.0025 0 rpy=0 0 0
- added joint L_pinky_intermediate_joint: type revolute, parent L_pinky_proximal_link, child L_pinky_intermediate_link, origin xyz=0.031532 -0.005451 0 rpy=0 0.00032164 -0.011403, axis 0 0 1, limit lower=-1.796 upper=0 effort=0 velocity=0, mimic joint=L_pinky_proximal_joint multiplier=0.975 offset=0
- added joint L_pinky_proximal_joint: type revolute, parent L_hand_base_link, child L_pinky_proximal_link, origin xyz=-0.028228 -0.0123 -0.094012 rpy=3.1416 1.4661 3.1416, axis 0 0 1, limit lower=-1.602 upper=0 effort=0 velocity=0
- added joint L_pinky_tip_joint: type fixed, parent L_pinky_intermediate_link, child L_pinky_tip_link, origin xyz=0.033 -0.0015 0 rpy=0 0 0
- added joint L_ring_intermediate_joint: type revolute, parent L_ring_proximal_link, child L_ring_intermediate_link, origin xyz=0.031531 -0.0054567 0.00025 rpy=0 0.00014037 -0.0025338, axis 0 0 1, limit lower=-1.798 upper=0 effort=0 velocity=0, mimic joint=L_ring_proximal_joint multiplier=0.975 offset=0
- added joint L_ring_proximal_joint: type revolute, parent L_hand_base_link, child L_ring_proximal_link, origin xyz=-0.010211 -0.0123 -0.095924 rpy=3.1416 1.5184 3.1416, axis 0 0 1, limit lower=-1.602 upper=0 effort=0 velocity=0
- added joint L_ring_tip_joint: type fixed, parent L_ring_intermediate_link, child L_ring_tip_link, origin xyz=0.0385 -0.0015 0 rpy=0 0 0
- added joint L_thumb_distal_joint: type revolute, parent L_thumb_proximal_pitch_link, child L_thumb_distal_link, origin xyz=0.061549 0.007464 0 rpy=0 1.7448E-05 -0.055652, axis 0 0 1, limit lower=0 upper=1.267 effort=0 velocity=0, mimic joint=L_thumb_proximal_pitch_joint multiplier=1.06 offset=0
- added joint L_thumb_proximal_pitch_joint: type revolute, parent L_thumb_proximal_yaw_link, child L_thumb_proximal_pitch_link, origin xyz=0.021749 -0.00016321 0 rpy=-1.5708 0 -0.0052052, axis 0 0 1, limit lower=0 upper=1.159 effort=0 velocity=0
- added joint L_thumb_proximal_yaw_joint: type revolute, parent L_hand_base_link, child L_thumb_proximal_yaw_link, origin xyz=0.022 -0.0155 -0.022992 rpy=0 0 0, axis 0 0 1, limit lower=-1.676 upper=0 effort=0 velocity=0
- added joint L_thumb_tip_joint: type fixed, parent L_thumb_distal_link, child L_thumb_tip_link, origin xyz=0.0305 -0.001 0 rpy=0 0 0
- added joint R_hand_base_joint: type fixed, parent right_end_effector_link, child R_hand_base_link, origin xyz=0 0 0 rpy=0 0 0
- added joint R_index_intermediate_joint: type revolute, parent R_index_proximal_link, child R_index_intermediate_link, origin xyz=0.031535 -0.0054349 0 rpy=0 0.00014037 -0.0012936, axis 0 0 1, limit lower=-1.791 upper=0 effort=0 velocity=0, mimic joint=R_index_proximal_joint multiplier=0.975 offset=0
- added joint R_index_proximal_joint: type revolute, parent R_hand_base_link, child R_index_proximal_link, origin xyz=0.026866 0.0123 -0.09399 rpy=3.1416 1.5184 0, axis 0 0 1, limit lower=-1.602 upper=0 effort=0 velocity=0
- added joint R_index_tip_joint: type fixed, parent R_index_intermediate_link, child R_index_tip_link, origin xyz=0.0390 -0.0020 0 rpy=0 0 0
- added joint R_middle_intermediate_joint: type revolute, parent R_middle_proximal_link, child R_middle_intermediate_link, origin xyz=0.031531 -0.0054597 0 rpy=0 0.00015517 0.007959, axis 0 0 1, limit lower=-1.791 upper=0 effort=0 velocity=0, mimic joint=R_middle_proximal_joint multiplier=0.975 offset=0
- added joint R_middle_proximal_joint: type revolute, parent R_hand_base_link, child R_middle_proximal_link, origin xyz=0.0085 0.0123 -0.096 rpy=3.1416 1.5708 0, axis 0 0 1, limit lower=-1.603 upper=0 effort=0 velocity=0
- added joint R_middle_tip_joint: type fixed, parent R_middle_intermediate_link, child R_middle_tip_link, origin xyz=0.047 -0.0025 0 rpy=0 0 0
- added joint R_pinky_intermediate_joint: type revolute, parent R_pinky_proximal_link, child R_pinky_intermediate_link, origin xyz=0.031474 -0.0057796 0 rpy=0 7.8504E-05 -0.030132, axis 0 0 1, limit lower=-1.796 upper=0 effort=0 velocity=0, mimic joint=R_pinky_proximal_joint multiplier=0.975 offset=0
- added joint R_pinky_proximal_joint: type revolute, parent R_hand_base_link, child R_pinky_proximal_link, origin xyz=-0.028223 0.0123 -0.093963 rpy=0 1.4661 3.1416, axis 0 0 1, limit lower=-1.602 upper=0 effort=0 velocity=0
- added joint R_pinky_tip_joint: type fixed, parent R_pinky_intermediate_link, child R_pinky_tip_link, origin xyz=0.033 -0.0015 0 rpy=0 0 0
- added joint R_ring_intermediate_joint: type revolute, parent R_ring_proximal_link, child R_ring_intermediate_link, origin xyz=0.031474 -0.0057806 0 rpy=0 0.00014037 -0.020997, axis 0 0 1, limit lower=-1.798 upper=0 effort=0 velocity=0, mimic joint=R_ring_proximal_joint multiplier=0.975 offset=0
- added joint R_ring_proximal_joint: type revolute, parent R_hand_base_link, child R_ring_proximal_link, origin xyz=-0.0099658 0.0123 -0.095888 rpy=0 1.5184 3.1416, axis 0 0 1, limit lower=-1.602 upper=0 effort=0 velocity=0
- added joint R_ring_tip_joint: type fixed, parent R_ring_intermediate_link, child R_ring_tip_link, origin xyz=0.0385 -0.0015 0 rpy=0 0 0
- added joint R_thumb_distal_joint: type revolute, parent R_thumb_proximal_pitch_link, child R_thumb_distal_link, origin xyz=0.061549 0.007464 0 rpy=0 1.7448E-05 -0.055652, axis 0 0 1, limit lower=0 upper=1.267 effort=0 velocity=0, mimic joint=R_thumb_proximal_pitch_joint multiplier=1.06 offset=0
- added joint R_thumb_proximal_pitch_joint: type revolute, parent R_thumb_proximal_yaw_link, child R_thumb_proximal_pitch_link, origin xyz=0.02175 -7.414E-05 0 rpy=1.5708 0 -0.0057076, axis 0 0 1, limit lower=0 upper=1.159 effort=0 velocity=0
- added joint R_thumb_proximal_yaw_joint: type revolute, parent R_hand_base_link, child R_thumb_proximal_yaw_link, origin xyz=0.022 0.0155 -0.022892 rpy=3.1416 0 0, axis 0 0 1, limit lower=-1.676 upper=0 effort=0 velocity=0
- added joint R_thumb_tip_joint: type fixed, parent R_thumb_distal_link, child R_thumb_tip_link, origin xyz=0.030 -0.0015 0 rpy=0 0 0
- joint camera_joint: origin xyz=0.090271 0 0.051067 rpy=0 0.2618 0 -> xyz=0.090296 0 0.05116 rpy=0 0.2618 0
- joint head_pitch_joint: limit lower=-0.50615 upper=0.50615 effort=17.4 velocity=9.21 -> lower=-0.5236 upper=0.1483 effort=17.4 velocity=9.21
- joint head_yaw_joint: limit lower=-1.3788 upper=1.3788 effort=17.4 velocity=9.21 -> lower=-1.3963 upper=1.3963 effort=17.4 velocity=9.21; origin xyz=0 0 0.18812 rpy=0 0 0 -> xyz=0.0077592 0 0.18812 rpy=0 0 0
- joint imu_joint: origin xyz=0 0 -0.069675 rpy=0 0 0 -> xyz=-0.005 0 -0.069675 rpy=0 0 0
- joint left_ankle_pitch_joint: limit lower=-0.76794 upper=0.76794 effort=59.4 velocity=16.76 -> lower=-0.7854 upper=0.7854 effort=59.4 velocity=16.76; origin xyz=0.019975 0 -0.425 rpy=0 0 0 -> xyz=0.020049 0 -0.425 rpy=0 0 0
- joint left_ankle_roll_joint: limit lower=-0.41888 upper=0.41888 effort=59.4 velocity=16.76 -> lower=-0.43633 upper=0.43633 effort=59.4 velocity=16.76; origin xyz=0 0 0 rpy=0 5.8728E-05 0 -> xyz=0 0 0 rpy=0 0 0
- joint left_elbow_pitch_joint: limit lower=-2.2515 upper=0.069813 effort=42.9 velocity=6.28 -> lower=-2.2689 upper=0.087266 effort=42.9 velocity=6.28; origin xyz=0.01643 0 -0.1445 rpy=0 0 0 -> xyz=0.01643 0 -0.1385 rpy=0 0 0
- joint left_end_effector_joint: origin xyz=-0.0013 0 -0.045 rpy=0 0 0 -> xyz=0 0 -0.049 rpy=0 0 0
- joint left_hip_pitch_joint: limit lower=-2.6005 upper=2.6005 effort=366 velocity=6.49 -> lower=-2.618 upper=2.618 effort=366 velocity=6.49; origin xyz=0 0.082061 -0.0071794 rpy=-0.087266 0 0 -> xyz=0 0.074191 -0.0064909 rpy=-0.087266 0 0
- joint left_hip_roll_joint: limit lower=-0.15708 upper=1.5533 effort=95.5 velocity=12.36 -> lower=-0.17453 upper=1.5708 effort=140.4 velocity=12.985; origin xyz=0 0.039 -0.015 rpy=0.087266 0 0 -> xyz=0 0.0479 -0.015 rpy=0.087266 0 0
- joint left_hip_yaw_joint: limit lower=-0.68068 upper=1.5533 effort=95.5 velocity=12.36 -> lower=-0.69813 upper=1.5708 effort=140.4 velocity=12.985; origin xyz=0.0052421 0.010464 -0.087239 rpy=0 0 0 -> xyz=0.0052421 0.010464 -0.093339 rpy=0 0 0
- joint left_knee_pitch_joint: limit lower=0 upper=2.3387 effort=366 velocity=6.49 -> lower=0 upper=2.3562 effort=366 velocity=6.49; origin xyz=0 0 -0.32099 rpy=0 0 0 -> xyz=0 0 -0.31499 rpy=0 0 0
- joint left_shoulder_pitch_joint: limit lower=-2.9496 upper=2.9496 effort=74.4 velocity=7.75 -> lower=-2.9671 upper=2.9671 effort=74.4 velocity=7.75; origin xyz=-0.025424 0.11818 0 rpy=0.53175 -0.16811 0.2775 -> xyz=-0.017665 0.11818 0 rpy=0.53175 -0.16811 0.2775
- joint left_shoulder_roll_joint: limit lower=-0.24435 upper=1.9024 effort=74.4 velocity=7.75 -> lower=-0.2618 upper=1.9199 effort=74.4 velocity=7.75
- joint left_shoulder_yaw_joint: limit lower=-1.8151 upper=1.8151 effort=42.9 velocity=6.28 -> lower=-1.8326 upper=1.8326 effort=42.9 velocity=6.28; origin xyz=0 -0.019582 -0.099541 rpy=-0.52348 0 0 -> xyz=0 -0.022594 -0.10473 rpy=-0.5236 0 0
- joint left_wrist_pitch_joint: limit lower=-0.7854 upper=0.95993 effort=17.4 velocity=9.2153 -> lower=-0.87266 upper=1.309 effort=17.4 velocity=9.2153; origin xyz=0 0 -0.1802 rpy=0 0 0 -> xyz=0 0 -0.18 rpy=0 0 0
- joint left_wrist_yaw_joint: limit lower=-1.8151 upper=1.8151 effort=42.9 velocity=6.28 -> lower=-1.8326 upper=1.8326 effort=42.9 velocity=6.28; origin xyz=-0.01643 0 -0.0498 rpy=0 0 0 -> xyz=-0.01643 0 -0.05 rpy=0 0 0
- joint right_ankle_pitch_joint: limit lower=-0.76794 upper=0.76794 effort=59.4 velocity=16.76 -> lower=-0.7854 upper=0.7854 effort=59.4 velocity=16.76
- joint right_ankle_roll_joint: limit lower=-0.41888 upper=0.41888 effort=59.4 velocity=16.76 -> lower=-0.43633 upper=0.43633 effort=59.4 velocity=16.76; origin xyz=0 0 0 rpy=0 7.6644E-05 0 -> xyz=0 0 0 rpy=0 0 0
- joint right_elbow_pitch_joint: limit lower=-2.2515 upper=0.069813 effort=42.9 velocity=6.28 -> lower=-2.2689 upper=0.087266 effort=42.9 velocity=6.28; origin xyz=0.01643 0 -0.1445 rpy=0 0 0 -> xyz=0.01643 0 -0.1385 rpy=0 0 0
- joint right_end_effector_joint: origin xyz=-0.0013 0 -0.045 rpy=0 0 0 -> xyz=0 0 -0.049 rpy=0 0 0
- joint right_hip_pitch_joint: limit lower=-2.6005 upper=2.6005 effort=366 velocity=6.49 -> lower=-2.618 upper=2.618 effort=366 velocity=6.49; origin xyz=0 -0.082061 -0.0071794 rpy=0.087266 0 0 -> xyz=0 -0.074191 -0.0064909 rpy=0.087266 0 0
- joint right_hip_roll_joint: limit lower=-1.5533 upper=0.15708 effort=95.5 velocity=12.36 -> lower=-1.5708 upper=0.17453 effort=140.4 velocity=12.985; origin xyz=0 -0.039 -0.015 rpy=-0.087266 0 0 -> xyz=0 -0.0479 -0.015 rpy=-0.087266 0 0
- joint right_hip_yaw_joint: limit lower=-1.5533 upper=0.68068 effort=95.5 velocity=12.36 -> lower=-1.5708 upper=0.69813 effort=140.4 velocity=12.985; origin xyz=0.0052421 -0.010464 -0.087239 rpy=0 0 0 -> xyz=0.0052421 -0.010464 -0.093339 rpy=0 0 0
- joint right_knee_pitch_joint: limit lower=0 upper=2.3387 effort=366 velocity=6.49 -> lower=0 upper=2.3562 effort=366 velocity=6.49; origin xyz=0 0 -0.32099 rpy=0 0 0 -> xyz=0 0 -0.31499 rpy=0 0 0
- joint right_shoulder_pitch_joint: limit lower=-2.9496 upper=2.9496 effort=74.4 velocity=7.75 -> lower=-2.9671 upper=2.9671 effort=74.4 velocity=7.75; origin xyz=-0.025424 -0.11819 0 rpy=-0.53175 -0.16811 -0.2775 -> xyz=-0.017665 -0.11819 0 rpy=-0.53175 -0.16811 -0.2775
- joint right_shoulder_roll_joint: limit lower=-1.9024 upper=0.24435 effort=74.4 velocity=7.75 -> lower=-1.9199 upper=0.2618 effort=74.4 velocity=7.75
- joint right_shoulder_yaw_joint: limit lower=-1.8151 upper=1.8151 effort=42.9 velocity=6.28 -> lower=-1.8326 upper=1.8326 effort=42.9 velocity=6.28; origin xyz=0 0.019582 -0.099541 rpy=0.52348 0 0 -> xyz=0 0.022594 -0.10473 rpy=0.5236 0 0
- joint right_wrist_pitch_joint: limit lower=-0.7854 upper=0.95993 effort=17.4 velocity=9.2153 -> lower=-0.87266 upper=1.309 effort=17.4 velocity=9.2153; origin xyz=0 0 -0.1802 rpy=0 0 0 -> xyz=0 0 -0.18 rpy=0 0 0
- joint right_wrist_roll_joint: origin xyz=0 0 0 rpy=0 0 0 -> xyz=0 -0.00049967 0 rpy=0 0 0
- joint right_wrist_yaw_joint: limit lower=-1.8151 upper=1.8151 effort=42.9 velocity=6.28 -> lower=-1.8326 upper=1.8326 effort=42.9 velocity=6.28; origin xyz=-0.01643 0 -0.0498 rpy=0 0 0 -> xyz=-0.01643 0 -0.05 rpy=0 0 0
- joint torso_joint: origin xyz=0.0077592 0 0.19798 rpy=0 0 0 -> xyz=0 0 0.19798 rpy=0 0 0
- joint waist_pitch_joint: limit lower=-0.20944 upper=0.50615 effort=108.6 velocity=14.77 -> lower=-0.20944 upper=0.5236 effort=108.6 velocity=14.77
- joint waist_roll_joint: limit lower=-0.15708 upper=0.15708 effort=108.6 velocity=14.77 -> lower=-0.17453 upper=0.17453 effort=108.6 velocity=14.77; origin xyz=-0.0077592 0 0.0491 rpy=0 0 0 -> xyz=0 0 0.0561 rpy=0 0 0
- joint waist_yaw_joint: limit lower=-2.6005 upper=2.6005 effort=95.47 velocity=12.36 -> lower=-2.618 upper=2.618 effort=140.4 velocity=12.985; origin xyz=0 0 0.14333 rpy=0 0 0 -> xyz=0 0 0.13633 rpy=0 0 0
