Commit message: Update gr3 urdf mesh path

File: openrd/urdf/fourier_gr3/gr3.urdf (robot description, URDF)
Before this commit: robot gr3v2_1_1, 71 links, 70 joints
Links:
- link L_hand_base_link: geometry collision mesh filename=../meshes/fourier_gr3/L_hand_base_link.STL; visual mesh filename=../meshes/fourier_gr3/L_hand_base_link.STL
- link L_index_intermediate_link: geometry collision mesh filename=../meshes/fourier_gr3/L_index_intermediate_link.STL; visual mesh filename=../meshes/fourier_gr3/L_index_intermediate_link.STL
- link L_index_proximal_link: geometry collision mesh filename=../meshes/fourier_gr3/L_index_proximal_link.STL; visual mesh filename=../meshes/fourier_gr3/L_index_proximal_link.STL
- link L_middle_intermediate_link: geometry collision mesh filename=../meshes/fourier_gr3/L_middle_intermediate_link.STL; visual mesh filename=../meshes/fourier_gr3/L_middle_intermediate_link.STL
- link L_middle_proximal_link: geometry collision mesh filename=../meshes/fourier_gr3/L_middle_proximal_link.STL; visual mesh filename=../meshes/fourier_gr3/L_middle_proximal_link.STL
- link L_pinky_intermediate_link: geometry collision mesh filename=../meshes/fourier_gr3/L_pinky_intermediate_link.STL; visual mesh filename=../meshes/fourier_gr3/L_pinky_intermediate_link.STL
- link L_pinky_proximal_link: geometry collision mesh filename=../meshes/fourier_gr3/L_pinky_proximal_link.STL; visual mesh filename=../meshes/fourier_gr3/L_pinky_proximal_link.STL
- link L_ring_intermediate_link: geometry collision mesh filename=../meshes/fourier_gr3/L_ring_intermediate_link.STL; visual mesh filename=../meshes/fourier_gr3/L_ring_intermediate_link.STL
- link L_ring_proximal_link: geometry collision mesh filename=../meshes/fourier_gr3/L_ring_proximal_link.STL; visual mesh filename=../meshes/fourier_gr3/L_ring_proximal_link.STL
- link L_thumb_distal_link: geometry collision mesh filename=../meshes/fourier_gr3/L_thumb_distal_link.STL; visual mesh filename=../meshes/fourier_gr3/L_thumb_distal_link.STL
- link L_thumb_proximal_pitch_link: geometry collision mesh filename=../meshes/fourier_gr3/L_thumb_proximal_pitch_link.STL; visual mesh filename=../meshes/fourier_gr3/L_thumb_proximal_pitch_link.STL
- link L_thumb_proximal_yaw_link: geometry collision mesh filename=../meshes/fourier_gr3/L_thumb_proximal_yaw_link.STL; visual mesh filename=../meshes/fourier_gr3/L_thumb_proximal_yaw_link.STL
- link R_hand_base_link: geometry collision mesh filename=../meshes/fourier_gr3/R_hand_base_link.STL; visual mesh filename=../meshes/fourier_gr3/R_hand_base_link.STL
- link R_index_intermediate_link: geometry collision mesh filename=../meshes/fourier_gr3/R_index_intermediate_link.STL; visual mesh filename=../meshes/fourier_gr3/R_index_intermediate_link.STL
- link R_index_proximal_link: geometry collision mesh filename=../meshes/fourier_gr3/R_index_proximal_link.STL; visual mesh filename=../meshes/fourier_gr3/R_index_proximal_link.STL
- link R_middle_intermediate_link: geometry collision mesh filename=../meshes/fourier_gr3/R_middle_intermediate_link.STL; visual mesh filename=../meshes/fourier_gr3/R_middle_intermediate_link.STL
- link R_middle_proximal_link: geometry collision mesh filename=../meshes/fourier_gr3/R_middle_proximal_link.STL; visual mesh filename=../meshes/fourier_gr3/R_middle_proximal_link.STL
- link R_pinky_intermediate_link: geometry collision mesh filename=../meshes/fourier_gr3/R_pinky_intermediate_link.STL; visual mesh filename=../meshes/fourier_gr3/R_pinky_intermediate_link.STL
- link R_pinky_proximal_link: geometry collision mesh filename=../meshes/fourier_gr3/R_pinky_proximal_link.STL; visual mesh filename=../meshes/fourier_gr3/R_pinky_proximal_link.STL
- link R_ring_intermediate_link: geometry collision mesh filename=../meshes/fourier_gr3/R_ring_intermediate_link.STL; visual mesh filename=../meshes/fourier_gr3/R_ring_intermediate_link.STL
- link R_ring_proximal_link: geometry collision mesh filename=../meshes/fourier_gr3/R_ring_proximal_link.STL; visual mesh filename=../meshes/fourier_gr3/R_ring_proximal_link.STL
- link R_thumb_distal_link: geometry collision mesh filename=../meshes/fourier_gr3/R_thumb_distal_link.STL; visual mesh filename=../meshes/fourier_gr3/R_thumb_distal_link.STL
- link R_thumb_proximal_pitch_link: geometry collision mesh filename=../meshes/fourier_gr3/R_thumb_proximal_pitch_link.STL; visual mesh filename=../meshes/fourier_gr3/R_thumb_proximal_pitch_link.STL
- link R_thumb_proximal_yaw_link: geometry collision mesh filename=../meshes/fourier_gr3/R_thumb_proximal_yaw_link.STL; visual mesh filename=../meshes/fourier_gr3/R_thumb_proximal_yaw_link.STL
